File: kicad/v2-beta/solar_cooker_v2.kicad_pcb (KiCad board)
At the start: 2 copper layers, 14 parts, among them J2 Conn_01x06_Pin, J3 Conn_01x14_Pin, J4 M20-9980346, SW2 SW_Push_Dual, U1 ATmega328P-P, U2 ATmega16U2-A, Y1 Resonator

Commit message: KiCad v2 update
Parts:
- added D1: 1N4148W, Diode_SMD:D_SOD-123, F.Cu at (108.3, 99.1)
- added J1: M20-9980346, 2x3 pin connector:HDRV6W64P254_2X3_762X508X868P, F.Cu at (144.8, 116.8)
- added J5: MUSB-05-X-B-SM-A, mini USB B:SAMTEC_MUSB-05-X-B-SM-A, F.Cu at (109.2, 88.9)
- added U3: LP2985-3.3, Package_TO_SOT_SMD:SOT-23-5, F.Cu at (107.8, 105.7)
