File: kicad/v2-beta/solar_cooker_v2.kicad_sch (KiCad schematic)
At the start: 14 parts, among them J2 Conn_01x06_Pin, J3 Conn_01x14_Pin, J4 M20-9980346, SW2 SW_Push_Dual, U1 ATmega328P-P, U2 ATmega16U2-A, Y1 Resonator

Commit message: KiCad v2 update
Parts:
- removed D2: ~, diode:LED-1206, symbol custom_components:diode
- added D1: 1N4148W, Diode_SMD:D_SOD-123, symbol Diode:1N4148W
- added J1: M20-9980346, HDRV6W64P254_2X3_762X508X868P, symbol M20-9980346:M20-9980346
- added J5: MUSB-05-X-B-SM-A, SAMTEC_MUSB-05-X-B-SM-A, symbol MUSB-05-X-B-SM-A:MUSB-05-X-B-SM-A
- added U3: LP2985-3.3, Package_TO_SOT_SMD:SOT-23-5, symbol Regulator_Linear:LP2985-3.3
- J2: Manufacturer Product Number (none) -> PPPC061LFBN-RC; Shop (none) -> Digi-Key
- J3: Manufacturer Product Number (none) -> PPPC141LFBN-RC; Shop (none) -> Digi-Key
- J4: Height 8.68 -> (none); Manufacturer Product Number (none) -> M20-9980346; Manufacturer_Name Harwin -> (none); Manufacturer_Part_Number M20-9980346 -> (none); Mouser Part Number 855-M20-9980346 -> (none); Mouser Price/Stock https://www.mouser.co.uk/ProductDetail/Harwin/M20-9980346?q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 -> (none)
- SW2: Manufacturer Product Number (none) -> SMT3-01-Z; Shop (none) -> Digi-Key
- U1: Manufacturer Product Number (none) -> ATMEGA328P-PN; Note (none) -> ED281DT Digi-Key; Shop (none) -> Digi-Key
- U2: Manufacturer Product Number (none) -> ATMEGA16U2-AUR; Shop (none) -> Digi-Key
- Y1: Manufacturer Product Number (none) -> CSTCE16M0V53-R0; Shop (none) -> Digi-Key
Connections:
- new net: J5.S1 (SHIELD), J5.S2 (SHIELD), J5.S3 (SHIELD), J5.S4 (SHIELD)
Other:
- moved on the sheet: U2

Commit message: kicad update
Parts:
- removed C4, C5: 100n, Capacitor_SMD:C_01005_0402Metric, symbol Device:C_Small
- removed D1: 1N4148W, Diode_SMD:D_SOD-123, symbol Diode:1N4148W
- removed J1, J4: M20-9980346, HDRV6W64P254_2X3_762X508X868P, symbol M20-9980346:M20-9980346
- removed J5: MUSB-05-X-B-SM-A, SAMTEC_MUSB-05-X-B-SM-A, symbol MUSB-05-X-B-SM-A:MUSB-05-X-B-SM-A
- removed R2: 1M, Resistor_SMD:R_01005_0402Metric, symbol Device:R_Small
- removed R3: 10k, Resistor_SMD:R_01005_0402Metric, symbol Device:R_Small
- removed SW2: SW_Push_Dual, push button:SMT3-01-Z, symbol Switch:SW_Push_Dual
- removed U1: ATmega328P-P, Package_DIP:DIP-28_W7.62mm, symbol MCU_Microchip_ATmega:ATmega328P-P
- removed U2: ATmega16U2-A, Package_QFP:TQFP-32_7x7mm_P0.8mm, symbol MCU_Microchip_ATmega:ATmega16U2-A
- removed Y1: Resonator, resonator:OSC_CSTCE16M0V53-R0, symbol Device:Resonator
Other:
- added sheet Arduino (arduino.kicad_sch)
- added sheet Sensors (sensors.kicad_sch)
- moved on the sheet: J2, J3, U3
