File: kicad/solar_cooker_v1.5.kicad_pcb (KiCad board)
At the start: 2 copper layers, 152.7 x 77.2 mm, 20 parts, among them J1 Pt100, J2 microSD, J3 Clock, J4 Pt100, J5 BME680, J6 GPS, J7 Pt100, J8 display, U1 anemometer, U2 AM2315C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

Commit message: order v2
Parts:
- J1, J4, J7: footprint custom_components:Pt100 -> custom_components:PT100
- J3: value Clock -> clock_module
- R1, R2: footprint Resistor_SMD:R_1206_3216Metric -> Resistor_SMD:R_1206_3216Metric_Pad1.30x1.75mm_HandSolder

Commit message: BOM generation update
now uses KiBoM
Parts:
- J1, J4, J7: footprint custom_components:PT100 -> custom_components:Pt100
Changed lines of the file:
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@@
     )
   )
-  (footprint "custom_components:PT100" (layer "F.Cu")
+  (footprint "custom_components:Pt100" (layer "F.Cu")
     (at 61.091 92.135 -90)
     (property "Description" "CONN RCPT 8POS 0.1 GOLD PCB")
@@
     (pad "8" thru_hole circle (at -8.89 -11.684 90) (size 1.65 1.65) (drill 1.1) (layers "*.Cu" "*.Mask")
       (net 107 "unconnected-(J1-RDY-Pad8)") (pinfunction "RDY") (pintype "input+no_connect"))
-    (group "" (id 623a924c-95bd-4c4a-954d-ff06fef4733c)
+    (group "" (id e78592cd-b16f-4062-bc88-1422561cbbe7)
       (members
-        1a0a85e8-d059-4fff-a2ad-1ae052af0887
-        1c071d07-fe9d-4313-8154-efd2b2125e9c
-        2c464b47-b808-45a4-a4ca-f2965185fbd2
-        54aa4a2f-ede6-4edf-8750-88a488e8fc8e
-        54f2213e-ca70-4be0-9575-5931968357a2
-        6a29bf8e-0365-41a3-b610-8276ffbf4660
-        8b35dafd-76a5-460b-90ed-2ed601655e29
-        a88dd608-1873-4bbd-8eb2-4a1e9cd3dbd2
+        04615028-6a03-4db4-9f69-1c4d2f3c172c
+        065145ce-60d5-4e41-b77f-25238be2c3c2
+        610780dd-2204-4dc1-b136-430da72b4f49
+        6e385cb4-66ee-48e2-9aec-bcb72355c4e1
+        ab1c4fa1-42b9-4b08-a81e-df3f2c13369a
+        cfb3c498-4508-4b87-96eb-0076e685eabe
+        f45d955e-f92d-4bc4-b2c5-ff8ee9ce039d
+        f9baf0e6-96a2-4839-b8cc-0246728baff0
       )
     )
@@
     )
   )
-  (footprint "custom_components:PT100" (layer "F.Cu")
+  (footprint "custom_components:Pt100" (layer "F.Cu")
     (at 61.091 118.635 -90)
     (property "Description" "CONN RCPT 8POS 0.1 GOLD PCB")
@@
     (pad "8" thru_hole circle (at -8.89 -11.684 90) (size 1.65 1.65) (drill 1.1) (layers "*.Cu" "*.Mask")
       (net 109 "unconnected-(J4-RDY-Pad8)") (pinfunction "RDY") (pintype "input+no_connect"))
-    (group "" (id 9cdb87b1-cade-4ee1-aacd-d3d379b8da1b)
+    (group "" (id c700da40-2614-46ed-94ba-ebaf6ab9062c)
       (members
-        1a65c976-29bf-4d48-8134-fc24732e6549
-        2da8ddbf-49d8-4902-aa19-935b273f0733
-        4a656f72-6fa9-4b00-95f0-1783a1f65459
-        58b57901-56f8-4292-b867-40067f6b0b82
-        880b8f20-4d36-4f95-abd7-45906cbc5aae
-        9e0fea17-0e3c-4cd7-b48d-e2dd07c8677c
-        e013d54c-3674-42b8-a767-d5726a943acc
-        ef7b9d50-94c0-4417-9a0a-ffec8dacac2a
+        3ab03805-94ce-40af-b0fe-d6f4ab7d1f72
+        757bcaad-34d7-4bf3-9587-ec6bdc4eaeff
+        845fef9f-08c1-4019-b332-5294a6de3be7
+        8a580078-826d-492d-92e8-3e218fa344a4
+        8a6f1042-0d8a-412a-a6ac-fe39ed7b5550
+        a2d57dcd-2d10-4ddd-9bd4-6841617e24e7
+        c4d33172-b038-4a21-a59d-dfd272934994
+        e4299b7b-9fe5-4f97-a1c5-e36001a484e0
       )
     )
@@
     (at 104.5375 125.475)
     (property "Description" "Slide Switch")
-    (property "MANUFACTURER" "E-switch")
-    (property "MAXIMUM_PACKAGE_HEIGHT" "13.59mm")
     (property "MPN" "500SSP1S2M2QEA")
     (property "Manufacturer" "E-switch")
-    (property "PARTREV" "C")
     (property "SPN" "EG5137-ND")
-    (property "STANDARD" "Manufacturer Recommendations")
     (property "Sheetfile" "solar_cooker_v1.5.kicad_sch")
     (property "Sheetname" "")
@@
       (net 2 "GND") (pinfunction "GND") (pintype "power_in"))
   )
-  (footprint "custom_components:PT100" (layer "F.Cu")
+  (footprint "custom_components:Pt100" (layer "F.Cu")
     (at 61.091 145.135 -90)
     (property "Description" "CONN RCPT 8POS 0.1 GOLD PCB")
@@
     (pad "8" thru_hole circle (at -8.89 -11.684 90) (size 1.65 1.65) (drill 1.1) (layers "*.Cu" "*.Mask")
       (net 111 "unconnected-(J7-RDY-Pad8)") (pinfunction "RDY") (pintype "input+no_connect"))
-    (group "" (id 2b7e7279-5595-4c14-b70f-8f0a6ea027ba)
+    (group "" (id 956d2f33-2ece-4764-8938-9ecefe2a81ab)
       (members
-        16f699d0-e08a-44ea-bb9e-cc283994e670
-        4a6e9ad7-c288-428b-bc8e-da6f220bc88a
-        5c172a42-b21d-41dd-8560-fc363ad501b5
-        789b38b7-4ffe-41a0-8b19-5d3414a1256c
-        895394ce-5641-482f-8b8b-a7738ae87a75
-        9346739d-b750-4daa-ade6-ba4f97eda9a8
-        d4cf0b51-76ea-4d4c-bd5e-3b9aedde2ada
-        ff87b4b4-371e-4cf7-bf13-ac5eb4d580d3
+        2965cd3c-e8ef-492d-8be0-b370e3950d16
+        5aebdf38-e4b2-4fb6-8b3c-5143e3a04986
+        67abf25f-e6e0-4f03-865f-ee2cfb850fc9
+        7fb78123-9ff9-4590-ae55-2c236c260e59
+        849c36e2-bda9-42a3-9793-1bd927da8f2b
+        986c1830-6a33-492c-865b-11ce87b5df7a
+        b4d09334-aa62-46e0-9ebb-d44d24feca45
+        efc8d213-50d4-4cb4-99b3-e00eb902674a
       )
     )
