File: kicad/solar_cooker.kicad_pcb (KiCad board)
At the start: 2 copper layers, 152.7 x 77.2 mm, 20 parts, among them J1 Pt100, J2 microSD, J3 clock, J4 Pt100, J5 BME680, J6 GPS, J7 Pt100, J8 display, U1 anemometer, U2 AM2315C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

Commit message: silkscreen update + schematic improvements
Changed lines of the file:
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@@
         (effects (font (size 1 1) (thickness 0.15)))
     )
-    (fp_text user "white" (at 2.6 7.119047 -90 unlocked) (layer "F.SilkS")
+    (fp_text user "white" (at 2.6 7.119047 270 unlocked) (layer "F.SilkS")
         (effects (font (size 1 1) (thickness 0.15)))
     )
@@
         (effects (font (size 1 1) (thickness 0.15)))
     )
-    (fp_text user "blue" (at 7.7 6.785714 -90 unlocked) (layer "F.SilkS")
+    (fp_text user "black" (at 7.7 7.190476 270 unlocked) (layer "F.SilkS")
         (effects (font (size 1 1) (thickness 0.15)))
     )
